Commit message: walks good forward!

File: src/quadruped_basics/urdf/quad.urdf.xacro (robot description, xacro)
@@ -32,5 +32,5 @@
     <origin xyz="0.069 0.098 -0.11469792884829269" rpy="-3.141592653589793 0 -3.141592653589793" />
     <axis xyz="0 0 1"/>
-    <limit effort="1000.0" lower="-1.57" upper="1.57" velocity="0.5"/>
+    <limit effort="1000.0"  velocity="0.5"/>
   </joint>
   <link name="cube5">
@@ -61,5 +61,5 @@
     <origin xyz="-0.048161324956420803 0.17705483565899827 0.019230531314252386" rpy="-1.570796326794897 0 1.570796326794897" />
     <axis xyz="0 0 1"/>
-    <limit effort="1000.0" lower="-1.57" upper="1.57" velocity="0.5"/>
+    <limit effort="1000.0" lower="-3.14" upper="3.14" velocity="0.5"/>
   </joint>
   <link name="cube9">
@@ -90,5 +90,5 @@
     <origin xyz="-0.1033382551226713 -0.0983866064663887 -0.11469792884829269" rpy="3.141592653589793 0 0" />
     <axis xyz="0 0 1"/>
-    <limit effort="1000.0" lower="-1.57" upper="1.57" velocity="0.5"/>
+    <limit effort="1000.0" lower="-3.14" upper="3.14" velocity="0.5"/>
   </joint>
   <link name="cube6">
@@ -119,5 +119,5 @@
     <origin xyz="-0.048161324956420803 0.17705483565899827 0.019230531314252386" rpy="-1.5707963267948966 0 1.5707963267948963" />
     <axis xyz="0 0 1"/>
-    <limit effort="1000.0" lower="-1.57" upper="1.57" velocity="0.5"/>
+    <limit effort="1000.0" lower="-3.14" upper="3.14" velocity="0.5"/>
   </joint>
   <link name="cube10">
@@ -148,5 +148,5 @@
     <origin xyz="0.09216405792838034 -0.0977373217828965 -0.11469792884829269" rpy="3.141592653589793 0 0" />
     <axis xyz="0 0 1"/>
-    <limit effort="1000.0" lower="-1.57" upper="1.57" velocity="0.5"/>
+    <limit effort="1000.0" lower="-3.14" upper="3.14" velocity="0.5"/>
   </joint>
   <link name="cube7">
@@ -177,5 +177,5 @@
     <origin xyz="0.04633851732690226 0.17705483565899827 0.019230531314252386" rpy="-1.5707963267948966 0 1.5707963267948963" />
     <axis xyz="0 0 1"/>
-    <limit effort="1000.0" lower="-1.57" upper="1.57" velocity="0.5"/>
+    <limit effort="1000.0" lower="-3.14" upper="3.14" velocity="0.5"/>
   </joint>
   <link name="cube11">
@@ -206,5 +206,5 @@
     <origin xyz="-0.10493619252487814 0.10058603880101953 -0.11469792884829269" rpy="-3.141592653589793 0 -3.141592653589793" />
     <axis xyz="0 0 1"/>
-    <limit effort="1000.0" lower="-1.57" upper="1.57" velocity="0.5"/>
+    <limit effort="1000.0" lower="-3.14" upper="3.14" velocity="0.5"/>
   </joint>
   <link name="cube8">
@@ -235,5 +235,5 @@
     <origin xyz="0.04633851732690226 0.17705483565899827 0.019230531314252386" rpy="-1.5707963267948966 0 1.5707963267948963" />
     <axis xyz="0 0 1"/>
-    <limit effort="1000.0" lower="-1.57" upper="1.57" velocity="0.5"/>
+    <limit effort="1000.0" lower="-3.14" upper="3.14" velocity="0.5"/>
   </joint>
   <link name="cube12">

Commit message: better turn and new map

File: src/quadruped_basics/urdf/quad.urdf.xacro (robot description, xacro)
@@ -273,6 +273,6 @@
     </collision>
     <inertial>
-      <mass value="0.05"/>
-      <inertia ixx="0.0001" ixy="0" ixz="0" iyy="0.0001" iyz="0" izz="0.0001"/>
+      <mass value="0.1"/>
+      <inertia ixx="0.001" ixy="0" ixz="0" iyy="0.001" iyz="0" izz="0.001"/>
     </inertial>
   </link>
