Commit message: Moving GZ simulation

File: src/quadruped_basics/urdf/quad.urdf.xacro (robot description, xacro)
@@ -23,5 +23,5 @@
     <inertial>
       <origin xyz="0 0 0" rpy="0 0 0" />
-      <mass value="1" />
+      <mass value="0.05" />
       <inertia ixx="0.16666666666666666" ixy="0" ixz="0" iyy="0.16666666666666666" iyz="0" izz="0.16666666666666666" />
     </inertial>
@@ -52,5 +52,5 @@
     <inertial>
       <origin xyz="0 0.103 0" rpy="0 0 0" />
-      <mass value="1" />
+      <mass value="0.05" />
       <inertia ixx="0.16666666666666666" ixy="0" ixz="0" iyy="0.16666666666666666" iyz="0" izz="0.16666666666666666" />
     </inertial>
@@ -81,5 +81,5 @@
     <inertial>
       <origin xyz="-2.127657382593146e-18 -0.125 0" rpy="0 0 0" />
-      <mass value="1" />
+      <mass value="0.05" />
       <inertia ixx="0.16666666666666666" ixy="0" ixz="0" iyy="0.16666666666666666" iyz="0" izz="0.16666666666666666" />
     </inertial>
@@ -110,5 +110,5 @@
     <inertial>
       <origin xyz="0 0.103 0" rpy="0 0 0" />
-      <mass value="1" />
+      <mass value="0.05" />
       <inertia ixx="0.16666666666666666" ixy="0" ixz="0" iyy="0.16666666666666666" iyz="0" izz="0.16666666666666666" />
     </inertial>
@@ -139,5 +139,5 @@
     <inertial>
       <origin xyz="-2.127657382593146e-18 -0.125 0" rpy="0 0 0" />
-      <mass value="1" />
+      <mass value="0.05" />
       <inertia ixx="0.16666666666666666" ixy="0" ixz="0" iyy="0.16666666666666666" iyz="0" izz="0.16666666666666666" />
     </inertial>
@@ -168,5 +168,5 @@
     <inertial>
       <origin xyz="0 0.103 0" rpy="0 0 0" />
-      <mass value="1" />
+      <mass value="0.05" />
       <inertia ixx="0.16666666666666666" ixy="0" ixz="0" iyy="0.16666666666666666" iyz="0" izz="0.16666666666666666" />
     </inertial>
@@ -197,5 +197,5 @@
     <inertial>
       <origin xyz="-2.127657382593146e-18 -0.125 0" rpy="0 0 0" />
-      <mass value="1" />
+      <mass value="0.05" />
       <inertia ixx="0.16666666666666666" ixy="0" ixz="0" iyy="0.16666666666666666" iyz="0" izz="0.16666666666666666" />
     </inertial>
@@ -226,5 +226,5 @@
     <inertial>
       <origin xyz="0 0.103 0" rpy="0 0 0" />
-      <mass value="1" />
+      <mass value="0.05" />
       <inertia ixx="0.16666666666666666" ixy="0" ixz="0" iyy="0.16666666666666666" iyz="0" izz="0.16666666666666666" />
     </inertial>
@@ -255,7 +255,77 @@
     <inertial>
       <origin xyz="-2.127657382593146e-18 -0.125 0" rpy="0 0 0" />
-      <mass value="1" />
-      <inertia ixx="0.16666666666666666" ixy="0" ixz="0" iyy="0.16666666666666666" iyz="0" izz="0.16666666666666666" />
-    </inertial>
-  </link>
+      <mass value="0.05" />
+      <inertia ixx="0.16666666666666666" ixy="0" ixz="0" iyy="0.16666666666666666" iyz="0" izz="0.16666666666666666" />
+    </inertial>
+  </link>
+  <ros2_control name="GazeboSimSystem" type="system">
+    <hardware>
+      <plugin>gz_ros2_control/GazeboSimSystem</plugin>
+    </hardware>
+    <joint name="base_link_to_cube5">
+      <command_interface name="position"/>
+      <state_interface name="position"/>
+    </joint>
+    <joint name="cube5_to_cube9">
+      <command_interface name="position"/>
+      <state_interface name="position"/>
+    </joint>
+    <joint name="base_link_to_cube6">
+      <command_interface name="position"/>
+      <state_interface name="position"/>
+    </joint>
+    <joint name="cube6_to_cube10">
+      <command_interface name="position"/>
+      <state_interface name="position"/>
+    </joint>
+    <joint name="base_link_to_cube7">
+      <command_interface name="position"/>
+      <state_interface name="position"/>
+    </joint>
+    <joint name="cube7_to_cube11">
+      <command_interface name="position"/>
+      <state_interface name="position"/>
+    </joint>
+    <joint name="base_link_to_cube8">
+      <command_interface name="position"/>
+      <state_interface name="position"/>
+    </joint>
+    <joint name="cube8_to_cube12">
+      <command_interface name="position"/>
+      <state_interface name="position"/>
+    </joint>
+  </ros2_control>
+  <gazebo reference="cube9">
+    <mu1>1.0</mu1>
+    <mu2>1.0</mu2>
+    <kp>1000000.0</kp>
+    <kd>100.0</kd>
+    <minDepth>0.001</minDepth>
+  </gazebo>
+  <gazebo reference="cube10">
+    <mu1>1.0</mu1>
+    <mu2>1.0</mu2>
+    <kp>1000000.0</kp>
+    <kd>100.0</kd>
+    <minDepth>0.001</minDepth>
+  </gazebo>
+  <gazebo reference="cube11">
+    <mu1>1.0</mu1>
+    <mu2>1.0</mu2>
+    <kp>1000000.0</kp>
+    <kd>100.0</kd>
+    <minDepth>0.001</minDepth>
+  </gazebo>
+  <gazebo reference="cube12">
+    <mu1>1.0</mu1>
+    <mu2>1.0</mu2>
+    <kp>1000000.0</kp>
+    <kd>100.0</kd>
+    <minDepth>0.001</minDepth>
+  </gazebo>
+  <gazebo>
+    <plugin filename="libgz_ros2_control-system.so" name="gz_ros2_control::GazeboSimROS2ControlPlugin">
+      <parameters>$(find quadruped_basics)/config/controllers.yaml</parameters>
+    </plugin>
+  </gazebo>
 </robot>

Commit message: added lidar

File: src/quadruped_basics/urdf/quad.urdf.xacro (robot description, xacro)
@@ -259,4 +259,46 @@
     </inertial>
   </link>
+  <joint name="belly_lidar_joint" type="fixed">
+    <parent link="base_link"/>
+    <child link="belly_lidar_link"/>
+    <origin xyz="0 0 -0.07" rpy="3.14159 0 0"/>
+  </joint>
+  <link name="belly_lidar_link">
+    <visual>
+      <geometry><cylinder radius="0.04" length="0.04"/></geometry>
+      <material name="black"><color rgba="0.1 0.1 0.1 1"/></material>
+    </visual>
+    <collision>
+      <geometry><cylinder radius="0.04" length="0.04"/></geometry>
+    </collision>
+    <inertial>
+      <mass value="0.05"/>
+      <inertia ixx="0.0001" ixy="0" ixz="0" iyy="0.0001" iyz="0" izz="0.0001"/>
+    </inertial>
+  </link>
+  <gazebo reference="belly_lidar_link">
+    <sensor name="belly_lidar" type="gpu_lidar">
+      <always_on>true</always_on>
+      <visualize>true</visualize>
+      <update_rate>10</update_rate>
+      <ray>
+        <scan>
+          <horizontal>
+            <samples>360</samples>
+            <resolution>1.0</resolution>
+            <min_angle>-3.14159</min_angle>
+            <max_angle>3.14159</max_angle>
+          </horizontal>
+        </scan>
+        <range>
+          <min>0.15</min>
+          <max>8.0</max>
+          <resolution>0.01</resolution>
+        </range>
+      </ray>
+      <topic>belly_scan</topic>
+      <gz_frame_id>belly_lidar_link</gz_frame_id>
+    </sensor>
+  </gazebo>
   <ros2_control name="GazeboSimSystem" type="system">
     <hardware>
@@ -329,3 +371,8 @@
     </plugin>
   </gazebo>
+  <gazebo>
+    <plugin filename="libgz-sim-sensors-system.so" name="gz::sim::systems::Sensors">
+      <render_engine>ogre2</render_engine>
+    </plugin>
+  </gazebo>
 </robot>

Commit message: added IMU to sim

File: src/quadruped_basics/urdf/quad.urdf.xacro (robot description, xacro)
@@ -259,4 +259,26 @@
     </inertial>
   </link>
+  <link name="imu_link">
+    <visual>
+      <geometry>
+        <box size="0.02 0.02 0.01"/>
+      </geometry>
+      <material name="red">
+        <color rgba="1.0 0.0 0.0 1.0"/>
+      </material>
+    </visual>
+  </link>
+  <joint name="imu_joint" type="fixed">
+    <parent link="base_link"/>
+    <child link="imu_link"/>
+    <origin xyz="0 0 0.05" rpy="0 0 0"/> </joint>
+  <gazebo reference="imu_link">
+    <sensor name="imu_sensor" type="imu">
+      <always_on>true</always_on>
+      <update_rate>50</update_rate>
+      <visualize>true</visualize>
+      <topic>imu</topic>
+    </sensor>
+  </gazebo>
   <joint name="belly_lidar_joint" type="fixed">
     <parent link="base_link"/>
@@ -376,3 +398,5 @@
     </plugin>
   </gazebo>
+  <plugin filename="gz-sim-imu-system" name="gz::sim::systems::Imu">
+  </plugin>
 </robot>
